File: 12f683MPPT.kicad_sch (KiCad schematic)
At the start: 51 parts, among them J1 Conn_01x01_Male, J2 Conn_01x01_Male, J3 Conn_01x01_Male, J4 Conn_01x01_Male, J5 Vin, J6 GND, J7 12V, Q1 BUK9511-55A127, Q2 BUK9511-55A127, Q3 2N2222A, Q4 2N2222A, Q5 2N2907A, SW1 SW_Push, U1 LM7805_TO220, U2 PIC12F683-IP, U3 LM358

Commit message: Hints on the capacity of the bootstrap capacitor C2.
Other:
- note added: "C2 = 0,47u : PWM>8kHz and FET Qg<50nS"
Changed lines of the file:
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@@
+		)
+	)
+	(text "C2 = 0,47u : PWM>8kHz and FET Qg<50nS"
+		(exclude_from_sim no)
+		(at 189.484 47.244 0)
+		(effects
+			(font
+				(size 1.27 1.27)
+			)
 		)
 	)
